Commit message: 2

File: src/turtlebot3_manipulation/turtlebot3_manipulation_description/gazebo/custom_four_wheel_base.gazebo.xacro (robot description, xacro)
@@ -9,6 +9,6 @@
     </gazebo>
     <gazebo reference="${prefix}wheel_left_link">
-      <mu1>10000.0</mu1>
-      <mu2>10000.0</mu2>
+      <mu1>10.0</mu1>
+      <mu2>1.0</mu2>
       <kp>500000.0</kp>
       <kd>10.0</kd>
@@ -19,6 +19,6 @@
     </gazebo>
     <gazebo reference="${prefix}wheel_right_link">
-      <mu1>10000.0</mu1>
-      <mu2>10000.0</mu2>
+      <mu1>10.0</mu1>
+      <mu2>1.0</mu2>
       <kp>500000.0</kp>
       <kd>10.0</kd>
@@ -29,6 +29,6 @@
     </gazebo>
     <gazebo reference="${prefix}caster_front_left_link">
-      <mu1>0.1</mu1>
-      <mu2>0.1</mu2>
+      <mu1>0.01</mu1>
+      <mu2>0.01</mu2>
       <kp>1000000.0</kp>
       <kd>100.0</kd>
@@ -38,6 +38,6 @@
     </gazebo>
     <gazebo reference="${prefix}caster_front_right_link">
-      <mu1>0.1</mu1>
-      <mu2>0.1</mu2>
+      <mu1>0.01</mu1>
+      <mu2>0.01</mu2>
       <kp>1000000.0</kp>
       <kd>100.0</kd>
@@ -58,5 +58,5 @@
         <wheel_diameter>0.135</wheel_diameter>
         <max_wheel_torque>20</max_wheel_torque>
-        <max_wheel_acceleration>10.0</max_wheel_acceleration>
+        <max_wheel_acceleration>1.0</max_wheel_acceleration>
         <publish_odom>true</publish_odom>
         <publish_odom_tf>true</publish_odom_tf>

File: src/turtlebot3_manipulation/turtlebot3_manipulation_description/urdf/custom_four_wheel_base.urdf.xacro (robot description, xacro)
@@ -15,5 +15,5 @@
     <link name="${prefix}base_link">
       <visual>
-        <origin xyz="0 0 0.03" rpy="0 0 0"/>
+        <origin xyz="0 0 0.05" rpy="0 0 0"/>
         <geometry>
           <box size="0.4 0.4 0.135"/>
@@ -24,5 +24,5 @@
       </visual>
       <collision>
-        <origin xyz="0 0 0.03" rpy="0 0 0"/>
+        <origin xyz="0 0 0.05" rpy="0 0 0"/>
         <geometry>
           <box size="0.4 0.4 0.135"/>
@@ -30,5 +30,5 @@
       </collision>
       <inertial>
-        <origin xyz="0 0 0.01" rpy="0 0 0"/>
+        <origin xyz="0.05 0 0.01" rpy="0 0 0"/>
         <mass value="5.0"/>
         <inertia ixx="0.2708" ixy="0.0" ixz="0.0"
@@ -41,5 +41,5 @@
       <parent link="${prefix}base_link"/>
       <child link="${prefix}wheel_left_link"/>
-      <origin xyz="-0.1 0.2 0" rpy="-1.57 0 0"/>
+      <origin xyz="-0.14 0.185 0" rpy="-1.57 0 0"/>
       <axis xyz="0 0 1"/>
     </joint>
@@ -72,5 +72,5 @@
       <parent link="${prefix}base_link"/>
       <child link="${prefix}wheel_right_link"/>
-      <origin xyz="-0.1 -0.2 0" rpy="-1.57 0 0"/>
+      <origin xyz="-0.14 -0.185 0" rpy="-1.57 0 0"/>
       <axis xyz="0 0 1"/>
     </joint>

Commit message: 2

File: src/turtlebot3_manipulation/turtlebot3_manipulation_description/gazebo/custom_four_wheel_base.gazebo.xacro (robot description, xacro)
@@ -116,5 +116,5 @@
         <visualize>${camera_visual}</visualize>
         <camera>
-            <horizontal_fov>1.085595</horizontal_fov>
+            <horizontal_fov>0.3</horizontal_fov>
             <image>
                 <width>640</width>

File: src/turtlebot3_manipulation/turtlebot3_manipulation_description/urdf/custom_four_wheel_base.urdf.xacro (robot description, xacro)
@@ -195,11 +195,17 @@
       <parent link="${prefix}base_link"/>
       <child link="${prefix}camera_link"/>
-      <origin xyz="0.2 0 0.1175" rpy="0 0 0"/>
+      <origin xyz="0.201 0 0.1" rpy="0 0 0"/>
     </joint>
     <link name="${prefix}camera_link">
-      <collision>
+      <visual>
         <origin xyz="0.005 0.011 0.013" rpy="0 0 0"/>
         <geometry>
-          <box size="0.015 0.030 0.027"/>
+          <box size="0.015 0.030 0.02"/>
+        </geometry>
+      </visual>
+      <collision>
+        <origin xyz="0.005 0.011 0.013" rpy="0 0 0"/>
+        <geometry>
+          <box size="0.015 0.030 0.02"/>
         </geometry>
       </collision>

Commit message: 4

File: src/turtlebot3_manipulation/turtlebot3_manipulation_description/gazebo/custom_four_wheel_base.gazebo.xacro (robot description, xacro)
@@ -9,20 +9,20 @@
     </gazebo>
     <gazebo reference="${prefix}wheel_left_link">
-      <mu1>10.0</mu1>
-      <mu2>1.0</mu2>
-      <kp>500000.0</kp>
-      <kd>10.0</kd>
+      <mu1>1.0</mu1>
+      <mu2>0.8</mu2>
+      <kp>350000.0</kp>
+      <kd>15.0</kd>
       <minDepth>0.001</minDepth>
-      <maxVel>0.1</maxVel>
+      <maxVel>0.3</maxVel>
       <fdir1>1 0 0</fdir1>
       <material>Gazebo/FlatBlack</material>
     </gazebo>
     <gazebo reference="${prefix}wheel_right_link">
-      <mu1>10.0</mu1>
-      <mu2>1.0</mu2>
-      <kp>500000.0</kp>
-      <kd>10.0</kd>
+      <mu1>1.0</mu1>
+      <mu2>0.8</mu2>
+      <kp>350000.0</kp>
+      <kd>15.0</kd>
       <minDepth>0.001</minDepth>
-      <maxVel>0.1</maxVel>
+      <maxVel>0.3</maxVel>
       <fdir1>1 0 0</fdir1>
       <material>Gazebo/FlatBlack</material>

File: src/turtlebot3_manipulation/turtlebot3_manipulation_description/urdf/custom_four_wheel_base.urdf.xacro (robot description, xacro)
@@ -30,6 +30,6 @@
       </collision>
       <inertial>
-        <origin xyz="0.05 0 0.01" rpy="0 0 0"/>
-        <mass value="5.0"/>
+        <origin xyz="-0.02 0 0.01" rpy="0 0 0"/>
+        <mass value="10.0"/>
         <inertia ixx="0.2708" ixy="0.0" ixz="0.0"
                  iyy="0.2708" iyz="0.0"

Commit message: 1

File: src/turtlebot3_manipulation/turtlebot3_manipulation_description/gazebo/custom_four_wheel_base.gazebo.xacro (robot description, xacro)
@@ -13,5 +13,5 @@
       <kp>350000.0</kp>
       <kd>15.0</kd>
-      <minDepth>0.001</minDepth>
+      <minDepth>0.002</minDepth>
       <maxVel>0.3</maxVel>
       <fdir1>1 0 0</fdir1>
@@ -23,5 +23,5 @@
       <kp>350000.0</kp>
       <kd>15.0</kd>
-      <minDepth>0.001</minDepth>
+      <minDepth>0.002</minDepth>
       <maxVel>0.3</maxVel>
       <fdir1>1 0 0</fdir1>
@@ -29,18 +29,18 @@
     </gazebo>
     <gazebo reference="${prefix}caster_front_left_link">
-      <mu1>0.01</mu1>
-      <mu2>0.01</mu2>
+      <mu1>0.001</mu1>
+      <mu2>0.001</mu2>
       <kp>1000000.0</kp>
       <kd>100.0</kd>
-      <minDepth>0.001</minDepth>
+      <minDepth>0.002</minDepth>
       <maxVel>1.0</maxVel>
       <material>Gazebo/FlatBlack</material>
     </gazebo>
     <gazebo reference="${prefix}caster_front_right_link">
-      <mu1>0.01</mu1>
-      <mu2>0.01</mu2>
+      <mu1>0.001</mu1>
+      <mu2>0.001</mu2>
       <kp>1000000.0</kp>
       <kd>100.0</kd>
-      <minDepth>0.001</minDepth>
+      <minDepth>0.002</minDepth>
       <maxVel>1.0</maxVel>
       <material>Gazebo/FlatBlack</material>
@@ -57,5 +57,5 @@
         <wheel_separation>0.3</wheel_separation>
         <wheel_diameter>0.135</wheel_diameter>
-        <max_wheel_torque>20</max_wheel_torque>
+        <max_wheel_torque>10</max_wheel_torque>
         <max_wheel_acceleration>1.0</max_wheel_acceleration>
         <publish_odom>true</publish_odom>

File: src/turtlebot3_manipulation/turtlebot3_manipulation_description/urdf/custom_four_wheel_base.urdf.xacro (robot description, xacro)
@@ -30,5 +30,5 @@
       </collision>
       <inertial>
-        <origin xyz="-0.02 0 0.01" rpy="0 0 0"/>
+        <origin xyz="0.0 0 0.01" rpy="0 0 0"/>
         <mass value="10.0"/>
         <inertia ixx="0.2708" ixy="0.0" ixz="0.0"

Commit message: 1

File: src/turtlebot3_manipulation/turtlebot3_manipulation_description/gazebo/custom_four_wheel_base.gazebo.xacro (robot description, xacro)
@@ -14,5 +14,5 @@
       <kd>15.0</kd>
       <minDepth>0.002</minDepth>
-      <maxVel>0.3</maxVel>
+      <maxVel>0.1</maxVel>
       <fdir1>1 0 0</fdir1>
       <material>Gazebo/FlatBlack</material>
@@ -24,5 +24,5 @@
       <kd>15.0</kd>
       <minDepth>0.002</minDepth>
-      <maxVel>0.3</maxVel>
+      <maxVel>0.1</maxVel>
       <fdir1>1 0 0</fdir1>
       <material>Gazebo/FlatBlack</material>
@@ -34,5 +34,5 @@
       <kd>100.0</kd>
       <minDepth>0.002</minDepth>
-      <maxVel>1.0</maxVel>
+      <maxVel>0.1</maxVel>
       <material>Gazebo/FlatBlack</material>
     </gazebo>
@@ -43,5 +43,5 @@
       <kd>100.0</kd>
       <minDepth>0.002</minDepth>
-      <maxVel>1.0</maxVel>
+      <maxVel>0.1</maxVel>
       <material>Gazebo/FlatBlack</material>
     </gazebo>
@@ -55,5 +55,5 @@
         <left_joint>wheel_left_joint</left_joint>
         <right_joint>wheel_right_joint</right_joint>
-        <wheel_separation>0.3</wheel_separation>
+        <wheel_separation>0.37</wheel_separation>
         <wheel_diameter>0.135</wheel_diameter>
         <max_wheel_torque>10</max_wheel_torque>

File: src/turtlebot3_manipulation/turtlebot3_manipulation_description/urdf/custom_four_wheel_base.urdf.xacro (robot description, xacro)
@@ -30,5 +30,5 @@
       </collision>
       <inertial>
-        <origin xyz="0.0 0 0.01" rpy="0 0 0"/>
+        <origin xyz="0.05 0 0.01" rpy="0 0 0"/>
         <mass value="10.0"/>
         <inertia ixx="0.2708" ixy="0.0" ixz="0.0"

File: src/turtlebot3_manipulation/turtlebot3_manipulation_description/urdf/fhbot.urdf.xacro (robot description, xacro)
@@ -13,5 +13,5 @@
   <!--导入底盘gazebo配置文件（物理属性，传感器，插件等） -->
   <xacro:include filename="$(find turtlebot3_manipulation_description)/gazebo/custom_four_wheel_base.gazebo.xacro" />
-  <!--根据参数prefix生成底盘及其gazebo插件 -->
+  <!--根据参数prefix生成底盘及其gazebo插件实例 -->
   <xacro:custom_four_wheel_base prefix="$(arg prefix)" />
   <xacro:custom_four_wheel_base_gazebo prefix="$(arg prefix)" />
