Commit message: 1

File: src/turtlebot3_manipulation/turtlebot3_manipulation_description/gazebo/custom_four_wheel_base.gazebo.xacro (robot description, xacro)
@@ -2,46 +2,58 @@
 <robot xmlns:xacro="http://ros.org/wiki/xacro">
   <xacro:macro name="custom_four_wheel_base_gazebo" params="prefix">
-  <xacro:property name="laser_visual"  value="true"/>
-  <xacro:property name="camera_visual" value="true"/>
-  <xacro:property name="imu_visual"    value="true"/>
+    <xacro:property name="laser_visual"  value="false"/>
+    <xacro:property name="camera_visual" value="false"/>
+    <xacro:property name="imu_visual"    value="true"/>
     <gazebo reference="${prefix}base_link">
-      <material>Gazebo/DarkGrey</material>
+      <material>Gazebo/Black</material>
+      <visual>
+        <transparency>0.5</transparency>
+      </visual>
+    </gazebo>
+    <gazebo reference="${prefix}center_of_mass_link">
+      <material>Gazebo/Red</material>
+    </gazebo>
+    <gazebo reference="${prefix}caster_connector_left_link">
+      <material>Gazebo/FlatBlack</material>
+    </gazebo>
+    <gazebo reference="${prefix}caster_connector_right_link">
+      <material>Gazebo/FlatBlack</material>
     </gazebo>
     <gazebo reference="${prefix}wheel_left_link">
-      <mu1>1.0</mu1>
+      <mu1>1</mu1>
       <mu2>0.8</mu2>
-      <kp>350000.0</kp>
-      <kd>15.0</kd>
-      <minDepth>0.002</minDepth>
-      <maxVel>0.1</maxVel>
+      <kp>200000.0</kp>
+      <kd>1000.0</kd>
+      <minDepth>0.001</minDepth>
+      <maxVel>0.2</maxVel>
       <fdir1>1 0 0</fdir1>
       <material>Gazebo/FlatBlack</material>
     </gazebo>
     <gazebo reference="${prefix}wheel_right_link">
-      <mu1>1.0</mu1>
+      <mu1>1</mu1>
       <mu2>0.8</mu2>
-      <kp>350000.0</kp>
-      <kd>15.0</kd>
-      <minDepth>0.002</minDepth>
-      <maxVel>0.1</maxVel>
+      <kp>200000.0</kp>
+      <kd>1000.0</kd>
+      <minDepth>0.001</minDepth>
+      <maxVel>0.2</maxVel>
       <fdir1>1 0 0</fdir1>
       <material>Gazebo/FlatBlack</material>
     </gazebo>
     <gazebo reference="${prefix}caster_front_left_link">
-      <mu1>0.001</mu1>
-      <mu2>0.001</mu2>
+      <mu1>0.1</mu1>
+      <mu2>0.05</mu2>
       <kp>1000000.0</kp>
       <kd>100.0</kd>
-      <minDepth>0.002</minDepth>
-      <maxVel>0.1</maxVel>
+      <minDepth>0.001</minDepth>
+      <maxVel>0.5</maxVel>
       <material>Gazebo/FlatBlack</material>
     </gazebo>
     <gazebo reference="${prefix}caster_front_right_link">
-      <mu1>0.001</mu1>
-      <mu2>0.001</mu2>
+      <mu1>0.1</mu1>
+      <mu2>0.05</mu2>
       <kp>1000000.0</kp>
       <kd>100.0</kd>
-      <minDepth>0.002</minDepth>
-      <maxVel>0.1</maxVel>
+      <minDepth>0.001</minDepth>
+      <maxVel>0.5</maxVel>
       <material>Gazebo/FlatBlack</material>
     </gazebo>
@@ -55,5 +67,5 @@
         <left_joint>wheel_left_joint</left_joint>
         <right_joint>wheel_right_joint</right_joint>
-        <wheel_separation>0.37</wheel_separation>
+        <wheel_separation>0.38</wheel_separation>
         <wheel_diameter>0.135</wheel_diameter>
         <max_wheel_torque>10</max_wheel_torque>

File: src/turtlebot3_manipulation/turtlebot3_manipulation_description/urdf/custom_four_wheel_base.urdf.xacro (robot description, xacro)
@@ -2,7 +2,22 @@
 <robot xmlns:xacro="http://www.ros.org/wiki/xacro">
   <xacro:macro name="custom_four_wheel_base" params="prefix">
-  <xacro:property
-  name="meshes_file_direction"
-  value="package://turtlebot3_manipulation_description/meshes/turtlebot3_waffle_pi"/>
+    <!-- 标量变量 -->
+    <xacro:property name="chassis_zero_height" value="0.09" />
+    <xacro:property name="chassis_length" value="0.41" />
+    <xacro:property name="chassis_width" value="0.4" />
+    <xacro:property name="chassis_height" value="0.2" />
+    <xacro:property name="driver_x_offset" value="-0.15" />
+    <xacro:property name="driver_y_offset" value="0.19" />
+    <xacro:property name="driver_radius" value="0.0675" />
+    <xacro:property name="caster_x_offset" value="0.15" />
+    <xacro:property name="caster_y_offset" value="0.08" />
+    <xacro:property name="caster_radius" value="0.025" />
+    <xacro:property name="chassis_heart_x_offset" value="0" />
+    <xacro:property name="chassis_heart_y_offset" value="0" />
+    <xacro:property name="chassis_heart_z_offset" value="-0.05" />
+    <xacro:property name="caster_z_offset" value="${driver_radius - caster_radius}" />
+    <xacro:property
+    name="meshes_file_direction"
+    value="package://turtlebot3_manipulation_description/meshes/turtlebot3_waffle_pi"/>
     <!-- Base footprint -->
     <link name="${prefix}base_footprint"/>
@@ -11,29 +26,44 @@
       <parent link="${prefix}base_footprint"/>
       <child link="${prefix}base_link"/>
-      <origin xyz="0.0 0.0 0.0675" rpy="0 0 0"/>
+      <origin xyz="0.0 0.0 ${driver_radius}" rpy="0 0 0"/>
     </joint>
     <link name="${prefix}base_link">
       <visual>
-        <origin xyz="0 0 0.05" rpy="0 0 0"/>
-        <geometry>
-          <box size="0.4 0.4 0.135"/>
-        </geometry>
-        <material name="grey">
-          <color rgba="0.5 0.5 0.5 1.0"/>
-        </material>
-      </visual>
-      <collision>
-        <origin xyz="0 0 0.05" rpy="0 0 0"/>
-        <geometry>
-          <box size="0.4 0.4 0.135"/>
-        </geometry>
-      </collision>
-      <inertial>
-        <origin xyz="0.05 0 0.01" rpy="0 0 0"/>
+        <origin xyz="0 0 ${chassis_zero_height+chassis_height/2-driver_radius}" rpy="0 0 0"/>
+        <geometry>
+          <box size="${chassis_length} ${chassis_width} ${chassis_height}"/>
+        </geometry>
+        <material name="transparent_black">
+          <color rgba="0 0 0 0.5"/>
+        </material>
+      </visual>
+      <collision>
+        <origin xyz="0 0 ${chassis_zero_height+chassis_height/2-driver_radius}" rpy="0 0 0"/>
+        <geometry>
+          <box size="${chassis_length} ${chassis_width} ${chassis_height}"/>
+        </geometry>
+      </collision>
+      <inertial>
+        <origin xyz="${chassis_heart_x_offset} ${chassis_heart_y_offset} ${chassis_zero_height+chassis_height/2-driver_radius+chassis_heart_z_offset}" rpy="0 0 0"/>
         <mass value="10.0"/>
         <inertia ixx="0.2708" ixy="0.0" ixz="0.0"
-                 iyy="0.2708" iyz="0.0"
-                 izz="0.2667"/>
-      </inertial>
+                  iyy="0.2708" iyz="0.0"
+                  izz="0.2667"/>
+      </inertial>
+    </link>
+    <joint name="${prefix}center_of_mass_joint" type="fixed">
+      <parent link="${prefix}base_link"/>
+      <child link="${prefix}center_of_mass_link"/>
+      <origin xyz="${chassis_heart_x_offset} ${chassis_heart_y_offset} ${chassis_zero_height+chassis_height/2-driver_radius+chassis_heart_z_offset}" rpy="0 0 0"/>
+    </joint>
+    <link name="${prefix}center_of_mass_link">
+      <visual>
+        <origin xyz="0 0 0" rpy="0 0 0"/>
+        <geometry>
+          <sphere radius="0.02"/>
+        </geometry>
+        <material name="red">
+        </material>
+      </visual>
     </link>
     <!-- Left drive wheel -->
@@ -41,5 +71,5 @@
       <parent link="${prefix}base_link"/>
       <child link="${prefix}wheel_left_link"/>
-      <origin xyz="-0.14 0.185 0" rpy="-1.57 0 0"/>
+      <origin xyz="${driver_x_offset} ${driver_y_offset} 0" rpy="-1.57 0 0"/>
       <axis xyz="0 0 1"/>
     </joint>
@@ -48,22 +78,20 @@
         <origin xyz="0 0 0" rpy="0 0 0"/>
         <geometry>
-          <cylinder radius="0.0675" length="0.03"/>
-        </geometry>
-        <material name="black">
-          <color rgba="0.0 0.0 0.0 1.0"/>
-        </material>
-      </visual>
-      <collision>
-        <origin xyz="0 0 0" rpy="0 0 0"/>
-        <geometry>
-          <cylinder radius="0.0675" length="0.03"/>
-        </geometry>
-      </collision>
-      <inertial>
-        <origin xyz="0 0 0" rpy="0 0 0"/>
-        <mass value="0.5"/>
+          <cylinder radius="${driver_radius}" length="0.03"/>
+        </geometry>
+        <material name="black"/>
+      </visual>
+      <collision>
+        <origin xyz="0 0 0" rpy="0 0 0"/>
+        <geometry>
+          <cylinder radius="${driver_radius}" length="0.03"/>
+        </geometry>
+      </collision>
+      <inertial>
+        <origin xyz="0 0 0" rpy="0 0 0"/>
+        <mass value="0.2"/>
         <inertia ixx="0.00114" ixy="0.0" ixz="0.0"
-                 iyy="0.00114" iyz="0.0"
-                 izz="0.00228"/>
+                  iyy="0.00114" iyz="0.0"
+                  izz="0.00228"/>
       </inertial>
     </link>
@@ -72,5 +100,5 @@
       <parent link="${prefix}base_link"/>
       <child link="${prefix}wheel_right_link"/>
-      <origin xyz="-0.14 -0.185 0" rpy="-1.57 0 0"/>
+      <origin xyz="${driver_x_offset} ${-driver_y_offset} 0" rpy="-1.57 0 0"/>
       <axis xyz="0 0 1"/>
     </joint>
@@ -79,82 +107,140 @@
         <origin xyz="0 0 0" rpy="0 0 0"/>
         <geometry>
-          <cylinder radius="0.0675" length="0.03"/>
-        </geometry>
-        <material name="black">
-          <color rgba="0.0 0.0 0.0 1.0"/>
-        </material>
-      </visual>
-      <collision>
-        <origin xyz="0 0 0" rpy="0 0 0"/>
-        <geometry>
-          <cylinder radius="0.0675" length="0.03"/>
-        </geometry>
-      </collision>
-      <inertial>
-        <origin xyz="0 0 0" rpy="0 0 0"/>
-        <mass value="0.5"/>
+          <cylinder radius="${driver_radius}" length="0.03"/>
+        </geometry>
+        <material name="black"/>
+      </visual>
+      <collision>
+        <origin xyz="0 0 0" rpy="0 0 0"/>
+        <geometry>
+          <cylinder radius="${driver_radius}" length="0.03"/>
+        </geometry>
+      </collision>
+      <inertial>
+        <origin xyz="0 0 0" rpy="0 0 0"/>
+        <mass value="0.2"/>
         <inertia ixx="0.00114" ixy="0.0" ixz="0.0"
-                 iyy="0.00114" iyz="0.0"
-                 izz="0.00228"/>
-      </inertial>
-    </link>
-    <!-- Front left caster wheel -->
+                  iyy="0.00114" iyz="0.0"
+                  izz="0.00228"/>
+      </inertial>
+    </link>
     <joint name="${prefix}caster_front_left_joint" type="fixed">
       <parent link="${prefix}base_link"/>
       <child link="${prefix}caster_front_left_link"/>
-      <origin xyz="0.15 0.1 -0.0425" rpy="0 0 0"/>
-    </joint>
-    <link name="${prefix}caster_front_left_link">
-      <visual>
-        <origin xyz="0 0 0" rpy="0 0 0"/>
-        <geometry>
-          <sphere radius="0.025"/>
-        </geometry>
-        <material name="black">
-          <color rgba="0.0 0.0 0.0 1.0"/>
-        </material>
-      </visual>
-      <collision>
-        <origin xyz="0 0 0" rpy="0 0 0"/>
-        <geometry>
-          <sphere radius="0.025"/>
-        </geometry>
-      </collision>
-      <inertial>
-        <origin xyz="0 0 0" rpy="0 0 0"/>
+      <origin xyz="${caster_x_offset} ${caster_y_offset} 0" rpy="0 0 0"/>
+    </joint>
+    <joint name="${prefix}caster_front_right_joint" type="fixed">
+      <parent link="${prefix}base_link"/>
+      <child link="${prefix}caster_front_right_link"/>
+      <origin xyz="${caster_x_offset} ${-caster_y_offset} 0" rpy="0 0 0"/>
+    </joint>
+    <joint name="${prefix}caster_connector_left_joint" type="fixed">
+      <parent link="${prefix}base_link"/>
+      <child link="${prefix}caster_connector_left_link"/>
+      <origin xyz="${caster_x_offset} ${caster_y_offset} 0" rpy="0 0 0"/>
+    </joint>
+    <joint name="${prefix}caster_connector_right_joint" type="fixed">
+      <parent link="${prefix}base_link"/>
+      <child link="${prefix}caster_connector_right_link"/>
+      <origin xyz="${caster_x_offset} ${-caster_y_offset} 0" rpy="0 0 0"/>
+    </joint>
+    <link name="${prefix}caster_connector_left_link">
+      <!-- 添加固定连杆 -->
+      <visual>
+        <origin xyz="0 0 ${chassis_zero_height/2-caster_z_offset}" rpy="0 0 0"/>
+        <geometry>
+          <cylinder radius="0.005" length="${chassis_zero_height-2*caster_radius}"/>
+        </geometry>
+        <material name="black">
+          <color rgba="0.0 0.0 0.0 1.0"/>
+        </material>
+      </visual>
+      <collision>
+        <origin xyz="0 0 ${chassis_zero_height/2-caster_z_offset}" rpy="0 0 0"/>
+        <geometry>
+          <cylinder radius="0.005" length="${chassis_zero_height-2*caster_radius}"/>
+        </geometry>
+      </collision>
+      <inertial>
+        <origin xyz="0 0 ${chassis_zero_height/2-caster_z_offset}" rpy="0 0 0"/>
         <mass value="0.1"/>
         <inertia ixx="0.00001" ixy="0.0" ixz="0.0"
-                 iyy="0.00001" iyz="0.0"
-                 izz="0.00001"/>
-      </inertial>
-    </link>
-    <!-- Front right caster wheel -->
-    <joint name="${prefix}caster_front_right_joint" type="fixed">
-      <parent link="${prefix}base_link"/>
-      <child link="${prefix}caster_front_right_link"/>
-      <origin xyz="0.15 -0.1 -0.0425" rpy="0 0 0"/>
-    </joint>
-    <link name="${prefix}caster_front_right_link">
-      <visual>
-        <origin xyz="0 0 0" rpy="0 0 0"/>
-        <geometry>
-          <sphere radius="0.025"/>
-        </geometry>
-        <material name="black">
-          <color rgba="0.0 0.0 0.0 1.0"/>
-        </material>
-      </visual>
-      <collision>
-        <origin xyz="0 0 0" rpy="0 0 0"/>
-        <geometry>
-          <sphere radius="0.025"/>
-        </geometry>
-      </collision>
-      <inertial>
-        <origin xyz="0 0 0" rpy="0 0 0"/>
+                  iyy="0.00001" iyz="0.0"
+                  izz="0.00001"/>
+      </inertial>
+    </link>
+    <link name="${prefix}caster_front_left_link">
+      <!-- 添加固定连杆 -->
+      <visual>
+        <origin xyz="0 0 ${-caster_z_offset}" rpy="0 0 0"/>
+        <geometry>
+          <sphere radius="${caster_radius}"/>
+        </geometry>
+        <material name="black">
+          <color rgba="0.0 0.0 0.0 1.0"/>
+        </material>
+      </visual>
+      <collision>
+        <origin xyz="0 0 ${-caster_z_offset}" rpy="0 0 0"/>
+        <geometry>
+          <sphere radius="${caster_radius}"/>
+        </geometry>
+      </collision>
+      <inertial>
+        <origin xyz="0 0 ${-caster_z_offset}" rpy="0 0 0"/>
         <mass value="0.1"/>
         <inertia ixx="0.00001" ixy="0.0" ixz="0.0"
-                 iyy="0.00001" iyz="0.0"
-                 izz="0.00001"/>
+                  iyy="0.00001" iyz="0.0"
+                  izz="0.00001"/>
+      </inertial>
+    </link>
+    <link name="${prefix}caster_connector_right_link">
+      <!-- 添加固定连杆 -->
+      <visual>
+        <origin xyz="0 0 ${chassis_zero_height/2-caster_z_offset}" rpy="0 0 0"/>
+        <geometry>
+          <cylinder radius="0.005" length="${chassis_zero_height-2*caster_radius}"/>
+        </geometry>
+        <material name="black">
+          <color rgba="0.0 0.0 0.0 1.0"/>
+        </material>
+      </visual>
+      <collision>
+        <origin xyz="0 0 ${chassis_zero_height/2-caster_z_offset}" rpy="0 0 0"/>
+        <geometry>
+          <cylinder radius="0.005" length="${chassis_zero_height-2*caster_radius}"/>
+        </geometry>
+      </collision>
+      <inertial>
+        <origin xyz="0 0 ${chassis_zero_height/2-caster_z_offset}" rpy="0 0 0"/>
+        <mass value="0.1"/>
+        <inertia ixx="0.00001" ixy="0.0" ixz="0.0"
+                  iyy="0.00001" iyz="0.0"
+                  izz="0.00001"/>
+      </inertial>
+    </link>
+    <link name="${prefix}caster_front_right_link">
+      <!-- 添加固定连杆 -->
+      <visual>
+        <origin xyz="0 0 ${-caster_z_offset}" rpy="0 0 0"/>
+        <geometry>
+          <sphere radius="${caster_radius}"/>
+        </geometry>
+        <material name="black">
+          <color rgba="0.0 0.0 0.0 1.0"/>
+        </material>
+      </visual>
+      <collision>
+        <origin xyz="0 0 ${-caster_z_offset}" rpy="0 0 0"/>
+        <geometry>
+          <sphere radius="${caster_radius}"/>
+        </geometry>
+      </collision>
+      <inertial>
+        <origin xyz="0 0 ${-caster_z_offset}" rpy="0 0 0"/>
+        <mass value="0.1"/>
+        <inertia ixx="0.00001" ixy="0.0" ixz="0.0"
+                  iyy="0.00001" iyz="0.0"
+                  izz="0.00001"/>
       </inertial>
     </link>
@@ -162,11 +248,21 @@
       <parent link="${prefix}base_link"/>
       <child link="${prefix}imu_link"/>
-      <origin xyz="0.0 0 0.068" rpy="0 0 0"/>
-    </joint>
-    <link name="${prefix}imu_link"/>
+      <origin xyz="0.0 0 ${chassis_zero_height-driver_radius-0.01}" rpy="0 0 0"/>
+    </joint>
+    <link name="${prefix}imu_link">
+      <visual>
+        <origin xyz="0 0 0" rpy="0 0 0"/>
+        <geometry>
+          <cylinder radius="0.03" length="0.02"/>
+        </geometry>
+        <material name="black">
+          <color rgba="0.0 0.0 0.0 1.0"/>
+        </material>
+      </visual>
+    </link>
     <joint name="${prefix}scan_joint" type="fixed">
       <parent link="${prefix}base_link"/>
       <child link="${prefix}base_scan"/>
-      <origin xyz="0.125 0 0.1375" rpy="0 0 0"/>
+      <origin xyz="${chassis_length/2-0.08} 0 ${chassis_zero_height-driver_radius+chassis_height+0.01}" rpy="0 0 0"/>
     </joint>
     <link name="${prefix}base_scan">
@@ -179,11 +275,11 @@
       </visual>
       <collision>
-        <origin xyz="0.015 0 -0.0065" rpy="0 0 0"/>
-        <geometry>
-          <cylinder length="0.0315" radius="0.055"/>
-        </geometry>
-      </collision>
-      <inertial>
-        <mass value="0.114" />
+        <origin xyz="0 0 0" rpy="0 0 0"/>
+        <geometry>
+          <mesh filename="${meshes_file_direction}/ladar.stl" scale="0.001 0.001 0.001"/>
+        </geometry>
+      </collision>
+      <inertial>
+        <mass value="0.1" />
         <origin xyz="0 0 0" />
         <inertia ixx="0.001" ixy="0.0" ixz="0.0"
@@ -195,17 +291,18 @@
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
File: src/turtlebot3_manipulation/turtlebot3_manipulation_description/urdf/fhbot.urdf.xacro (robot description, xacro)
@@ -8,5 +8,5 @@
   <xacro:arg name="fake_sensor_commands" default="false" />
   <!--导入材料定义文件 -->
-  <xacro:include filename="$(find turtlebot3_manipulation_description)/gazebo/materials.xacro" />
+  <xacro:include filename="$(find turtlebot3_manipulation_description)/urdf/materials.xacro" />
   <!--导入底盘urdf模型 -->
   <xacro:include filename="$(find turtlebot3_manipulation_description)/urdf/custom_four_wheel_base.urdf.xacro" />
@@ -42,5 +42,5 @@
   <gazebo>
     <plugin name="gazebo_ros2_control" filename="libgazebo_ros2_control.so">
-      <parameters>$(find turtlebot3_manipulation_bringup)/config/gazebo_controller_manager.yaml</parameters>
+      <parameters>$(find turtlebot3_manipulation_bringup)/config/gazebo_fhbot_ctrlmanager.yaml</parameters>
     </plugin>
   </gazebo>

File: src/turtlebot3_manipulation/turtlebot3_manipulation_description/urdf/materials.xacro (robot description, xacro)
@@ -5,4 +5,7 @@
 -->
 <robot>
+  <material name="transparent_grey">
+    <color rgba="0.5 0.5 0.5 0.5"/>
+  </material>
   <material name="black">
     <color rgba="0.0 0.0 0.0 1.0"/>

Commit message: 1

File: src/turtlebot3_manipulation/turtlebot3_manipulation_description/gazebo/custom_four_wheel_base.gazebo.xacro (robot description, xacro)
@@ -2,6 +2,6 @@
 <robot xmlns:xacro="http://ros.org/wiki/xacro">
   <xacro:macro name="custom_four_wheel_base_gazebo" params="prefix">
-    <xacro:property name="laser_visual"  value="false"/>
-    <xacro:property name="camera_visual" value="false"/>
+    <xacro:property name="laser_visual"  value="true"/>
+    <xacro:property name="camera_visual" value="true"/>
     <xacro:property name="imu_visual"    value="true"/>
     <gazebo reference="${prefix}base_link">
@@ -21,20 +21,20 @@
     </gazebo>
     <gazebo reference="${prefix}wheel_left_link">
-      <mu1>1</mu1>
-      <mu2>0.8</mu2>
-      <kp>200000.0</kp>
-      <kd>1000.0</kd>
+      <mu1>0.8</mu1>
+      <mu2>0.6</mu2>
+      <kp>300000.0</kp>
+      <kd>3000.0</kd>
       <minDepth>0.001</minDepth>
-      <maxVel>0.2</maxVel>
+      <maxVel>1.0</maxVel>
       <fdir1>1 0 0</fdir1>
       <material>Gazebo/FlatBlack</material>
     </gazebo>
     <gazebo reference="${prefix}wheel_right_link">
-      <mu1>1</mu1>
-      <mu2>0.8</mu2>
-      <kp>200000.0</kp>
-      <kd>1000.0</kd>
+      <mu1>0.8</mu1>
+      <mu2>0.6</mu2>
+      <kp>300000.0</kp>
+      <kd>3000.0</kd>
       <minDepth>0.001</minDepth>
-      <maxVel>0.2</maxVel>
+      <maxVel>1.0</maxVel>
       <fdir1>1 0 0</fdir1>
       <material>Gazebo/FlatBlack</material>
@@ -42,18 +42,18 @@
     <gazebo reference="${prefix}caster_front_left_link">
       <mu1>0.1</mu1>
-      <mu2>0.05</mu2>
+      <mu2>0.1</mu2>
       <kp>1000000.0</kp>
-      <kd>100.0</kd>
+      <kd>10000.0</kd>
       <minDepth>0.001</minDepth>
-      <maxVel>0.5</maxVel>
+      <maxVel>2.0</maxVel>
       <material>Gazebo/FlatBlack</material>
     </gazebo>
     <gazebo reference="${prefix}caster_front_right_link">
       <mu1>0.1</mu1>
-      <mu2>0.05</mu2>
+      <mu2>0.1</mu2>
       <kp>1000000.0</kp>
-      <kd>100.0</kd>
+      <kd>10000.0</kd>
       <minDepth>0.001</minDepth>
-      <maxVel>0.5</maxVel>
+      <maxVel>2.0</maxVel>
       <material>Gazebo/FlatBlack</material>
     </gazebo>
@@ -128,5 +128,5 @@
         <visualize>${camera_visual}</visualize>
         <camera>
-            <horizontal_fov>0.3</horizontal_fov>
+            <horizontal_fov>1.5</horizontal_fov>
             <image>
                 <width>640</width>
@@ -153,4 +153,5 @@
             <remapping>camera_info:=camera_info</remapping>
           </ros>
+          <fov_update>true</fov_update> <!-- 启用FOV更新支持 -->
         </plugin>
       </sensor>
