Commit message: sensors

File: src/turtlebot3_manipulation/turtlebot3_manipulation_description/gazebo/custom_four_wheel_base.gazebo.xacro (robot description, xacro)
@@ -2,7 +2,22 @@
 <robot xmlns:xacro="http://ros.org/wiki/xacro">
   <xacro:macro name="custom_four_wheel_base_gazebo" params="prefix">
-    <xacro:property name="laser_visual"  value="true"/>
-    <xacro:property name="camera_visual" value="true"/>
-    <xacro:property name="imu_visual"    value="true"/>
+    <xacro:property name="laser_visual"      value="false"/>
+    <xacro:property name="imu_visual"        value="true"/>
+    <xacro:property name="line_laser_visual" value="true"/>
+    <xacro:property name="tof_camera_visual" value="true"/>
+    <xacro:property name="base_laser_samples" value="360"/>
+    <xacro:property name="base_laser_rate" value="5"/>
+    <xacro:property name="base_laser_radius_min" value="0.12"/>
+    <xacro:property name="base_laser_radius_max" value="5"/>
+    <xacro:property name="line_laser_samples" value="148"/>
+    <xacro:property name="line_laser_rate" value="10"/>
+    <xacro:property name="line_laser_radius_min" value="0.07"/>
+    <xacro:property name="line_laser_radius_max" value="1"/>
+    <xacro:property name="side_laser_ang_min" value="-0.6"/>
+    <xacro:property name="side_laser_ang_max" value="0.8"/>
+    <xacro:property name="tof_camera_hfov" value="1.8"/>
+    <xacro:property name="tof_camera_rate" value="30"/>
+    <xacro:property name="tof_camera_radius_min" value="0.05"/>
+    <xacro:property name="tof_camera_radius_max" value="2"/>
     <gazebo reference="${prefix}base_link">
       <material>Gazebo/Black</material>
@@ -39,4 +54,27 @@
       <fdir1>1 0 0</fdir1>
       <material>Gazebo/FlatBlack</material>
+    </gazebo>
+    <!-- 编码器材料 -->
+    <gazebo reference="${prefix}wheel_left_encoder_link">
+      <material>Gazebo/Yellow</material>
+    </gazebo>
+    <gazebo reference="${prefix}wheel_right_encoder_link">
+      <material>Gazebo/Yellow</material>
+    </gazebo>
+    <gazebo>
+      <plugin name="joint_state_publisher" filename="libgazebo_ros_joint_state_publisher.so">
+        <ros>
+          <namespace></namespace>
+          <remapping>joint_states:=wheel_encoder_states</remapping>
+        </ros>
+        <update_rate>100.0</update_rate>
+        <joint_name>${prefix}wheel_left_joint</joint_name>
+        <joint_name>${prefix}wheel_right_joint</joint_name>
+        <position_noise>
+          <type>gaussian</type>
+          <mean>0.0</mean>
+          <stddev>0.001</stddev>  <!-- 编码器位置精度很高，噪声很小 -->
+        </position_noise>
+      </plugin>
     </gazebo>
     <gazebo reference="${prefix}caster_front_left_link">
@@ -84,18 +122,60 @@
         <update_rate>100.0</update_rate>
         <visualize>${imu_visual}</visualize>
+        <!-- IMU噪声配置 -->
+        <imu>
+          <angular_velocity>
+            <x>
+              <noise type="gaussian">
+                <mean>0.0</mean>
+                <stddev>0.002</stddev>
+              </noise>
+            </x>
+            <y>
+              <noise type="gaussian">
+                <mean>0.0</mean>
+                <stddev>0.002</stddev>
+              </noise>
+            </y>
+            <z>
+              <noise type="gaussian">
+                <mean>0.0</mean>
+                <stddev>0.002</stddev>
+              </noise>
+            </z>
+          </angular_velocity>
+          <linear_acceleration>
+            <x>
+              <noise type="gaussian">
+                <mean>0.0</mean>
+                <stddev>0.01</stddev>
+              </noise>
+            </x>
+            <y>
+              <noise type="gaussian">
+                <mean>0.0</mean>
+                <stddev>0.01</stddev>
+              </noise>
+            </y>
+            <z>
+              <noise type="gaussian">
+                <mean>0.0</mean>
+                <stddev>0.01</stddev>
+              </noise>
+            </z>
+          </linear_acceleration>
+        </imu>
       </sensor>
     </gazebo>
     <gazebo reference="${prefix}base_scan">
       <material>Gazebo/FlatBlack</material>
-      <sensor type="ray" name="lds_lfcd_sensor">
-        <pose>0 0 0 0 0 0</pose>
-        <always_on>true</always_on>
-        <update_rate>5.0</update_rate>
+      <sensor type="ray" name="base_scan">
+        <pose>0 0 0 0 0 0</pose>
+        <always_on>true</always_on>
+        <update_rate>${base_laser_rate}</update_rate>
         <visualize>${laser_visual}</visualize>
         <ray>
           <scan>
             <horizontal>
-              <samples>360</samples>
-              <resolution>1</resolution>
+              <samples>${base_laser_samples}</samples>
               <min_angle>0.0</min_angle>
               <max_angle>6.28319</max_angle>
@@ -103,7 +183,6 @@
           </scan>
           <range>
-            <min>0.120</min>
-            <max>3.5</max>
-            <resolution>0.015</resolution>
+            <min>${base_laser_radius_min}</min>
+            <max>${base_laser_radius_max}</max>
           </range>
           <noise>
@@ -116,5 +195,5 @@
           <ros>
             <namespace></namespace>
-            <remapping>~/out:=scan</remapping>
+            <remapping>~/out:=base_scan</remapping>
           </ros>
           <output_type>sensor_msgs/LaserScan</output_type>
@@ -122,36 +201,175 @@
       </sensor>
     </gazebo>
-    <gazebo reference="${prefix}camera_rgb_frame">
-      <sensor type="camera" name="pi_camera">
-        <update_rate>30</update_rate>
-        <always_on>true</always_on>
-        <visualize>${camera_visual}</visualize>
-        <camera>
-            <horizontal_fov>1.5</horizontal_fov>
-            <image>
-                <width>640</width>
-                <height>480</height>
-                <format>R8G8B8</format>
-            </image>
-            <clip>
-                <near>0.03</near>
-                <far>100</far>
-            </clip>
-            <noise>
-              <type>gaussian</type>
-              <!-- Noise is sampled independently per pixel on each frame.
-                  That pixel's noise value is added to each of its color
-                  channels, which at that point lie in the range [0,1]. -->
-              <mean>0.0</mean>
-              <stddev>0.007</stddev>
-            </noise>
-        </camera>
-        <plugin name="camera_controller" filename="libgazebo_ros_camera.so">
+    <!-- 左线激光传感器配置 - 添加适度噪声 -->
+    <gazebo reference="${prefix}line_laser_left">
+      <material>Gazebo/Red</material>
+      <sensor name="line_laser_left" type="ray">
+        <pose>0 0 0 0 0 0</pose>
+        <always_on>true</always_on>
+        <update_rate>${line_laser_rate}</update_rate>
+        <visualize>${line_laser_visual}</visualize>
+        <ray>
+          <scan>
+            <vertical>
+              <samples>1</samples>
+              <resolution>1.0</resolution>
+              <min_angle>0</min_angle>
+              <max_angle>0</max_angle>
+            </vertical>
+            <horizontal>
+              <samples>${line_laser_samples}</samples>
+              <min_angle>${side_laser_ang_min}</min_angle>
+              <max_angle>${side_laser_ang_max}</max_angle>
+            </horizontal>
+          </scan>
+          <range>
+            <min>${line_laser_radius_min}</min>
+            <max>${line_laser_radius_max}</max>
+          </range>
+          <!-- 添加噪声模型 -->
+          <noise>
+            <type>gaussian</type>
+            <!-- ±0.5cm的距离噪声 -->
+            <mean>0.0</mean>
+            <stddev>0.005</stddev> <!-- 0.5厘米标准差 -->
+          </noise>
+        </ray>
+        <plugin name="gazebo_ros_line_lazer_left_controller" filename="libgazebo_ros_ray_sensor.so">
           <ros>
             <namespace></namespace>
-            <remapping>image_raw:=image_raw</remapping>
-            <remapping>camera_info:=camera_info</remapping>
+            <remapping>~/out:=line_scan_left</remapping>
           </ros>
-          <fov_update>true</fov_update> <!-- 启用FOV更新支持 -->
+          <output_type>sensor_msgs/LaserScan</output_type>
+        </plugin>
+      </sensor>
+    </gazebo>
+    <!-- 中线激光传感器配置 - 添加适度噪声 -->
+    <gazebo reference="${prefix}line_laser_mid">
+      <material>Gazebo/Red</material>
+      <sensor name="line_laser_mid" type="ray">
+        <pose>0 0 0 0 0 0</pose>
+        <always_on>true</always_on>
+        <update_rate>${line_laser_rate}</update_rate>
+        <visualize>${line_laser_visual}</visualize>
+        <ray>
+          <scan>
+            <vertical>
+              <samples>1</samples>
+              <resolution>1.0</resolution>
+              <min_angle>0</min_angle>
+              <max_angle>0</max_angle>
+            </vertical>
+            <horizontal>
+              <samples>${line_laser_samples}</samples>
+              <min_angle>${(side_laser_ang_min-side_laser_ang_max)/2}</min_angle>
+              <max_angle>${(side_laser_ang_max-side_laser_ang_min)/2}</max_angle>
+            </horizontal>
+          </scan>
+          <range>
+            <min>${line_laser_radius_min}</min>
+            <max>${line_laser_radius_max}</max>
+          </range>
+          <!-- 添加噪声模型 -->
+          <noise>
+            <type>gaussian</type>
+            <!-- ±0.5cm的距离噪声 -->
+            <mean>0.0</mean>
+            <stddev>0.005</stddev> <!-- 0.5厘米标准差 -->
+          </noise>
+        </ray>
+        <plugin name="gazebo_ros_line_lazer_mid_controller" filename="libgazebo_ros_ray_sensor.so">
+          <ros>
+            <namespace></namespace>
+            <remapping>~/out:=line_scan_mid</remapping>
+          </ros>
+          <output_type>sensor_msgs/LaserScan</output_type>
+        </plugin>
+      </sensor>
+    </gazebo>
+    <!-- 右线激光传感器配置 - 添加适度噪声 -->
+    <gazebo reference="${prefix}line_laser_right">
+      <material>Gazebo/Red</material>
+      <sensor name="line_laser_right" type="ray">
+        <pose>0 0 0 0 0 0</pose>
+        <always_on>true</always_on>
+        <update_rate>${line_laser_rate}</update_rate>
+        <visualize>${line_laser_visual}</visualize>
+        <ray>
+          <scan>
+            <vertical>
+              <samples>1</samples>
+              <resolution>1.0</resolution>
+              <min_angle>0</min_angle>
+              <max_angle>0</max_angle>
+            </vertical>
+            <horizontal>
+              <samples>${line_laser_samples}</samples>
+              <min_angle>${side_laser_ang_min}</min_angle>
+              <max_angle>${side_laser_ang_max}</max_angle>
+            </horizontal>
+          </scan>
+          <range>
+            <min>${line_laser_radius_min}</min>
+            <max>${line_laser_radius_max}</max>
+          </range>
+          <!-- 添加噪声模型 -->
+          <noise>
+            <type>gaussian</type>
+            <!-- ±0.5cm的距离噪声 -->
+            <mean>0.0</mean>
+            <stddev>0.005</stddev> <!-- 0.5厘米标准差 -->
+          </noise>
+        </ray>
+        <plugin name="gazebo_ros_line_lazer_right_controller" filename="libgazebo_ros_ray_sensor.so">
+          <ros>
+            <namespace></namespace>
+            <remapping>~/out:=line_scan_right</remapping>
+          </ros>
+          <output_type>sensor_msgs/LaserScan</output_type>
+        </plugin>
+      </sensor>
+    </gazebo>
+    <!-- 3D ToF深度相机配置 -->
+    <gazebo reference="${prefix}tof_camera">
+      <material>Gazebo/Blue</material>
+      <sensor type="depth" name="tof_camera">
+        <pose>0 0 0 0 0 0</pose>
+        <always_on>true</always_on>
+        <update_rate>${tof_camera_rate}</update_rate>
+        <visualize>${tof_camera_visual}</visualize>
+        <camera name="camera">
+          <horizontal_fov>${tof_camera_hfov}</horizontal_fov>
+          <image>
+            <width>800</width>
+            <height>600</height>
+            <format>R8G8B8</format>
+          </image>
+          <distortion>
+            <k1>0.0</k1>
+            <k2>0.0</k2>
+            <k3>0.0</k3>
+            <p1>0.0</p1>
+            <p2>0.0</p2>
+            <center>0.5 0.5</center>
+          </distortion>
+          <!-- 添加噪声配置 -->
+          <noise>
+            <type>gaussian</type>
+            <mean>0.0</mean>
+            <stddev>0.01</stddev>
+          </noise>
+          <clip>
+            <near>${tof_camera_radius_min}</near>
+            <far>${tof_camera_radius_max}</far>
+          </clip>
+          <link name = "${prefix}camera_optical_link"> </link>
+          <joint name="${prefix}camera_optical_joint" type="fixed">
+            <parent link="${prefix}tof_camera"/>
+            <child link="${prefix}camera_optical_link"/>
+            <origin xyz="0 0 0" rpy="-1.57 0 -1.57"/>
+          </joint>
+        </camera>
+        <plugin name="depth_camera" filename="libgazebo_ros_camera.so">
+          <frame_name>${prefix}camera_optical_link</frame_name>
         </plugin>
       </sensor>

File: src/turtlebot3_manipulation/turtlebot3_manipulation_description/ros2_control/fhbot_system.ros2_control.xacro (robot description, xacro)
@@ -88,5 +88,5 @@
         </state_interface>
       </sensor>
-      <sensor name="battery">
+      <!-- <sensor name="battery">
         <state_interface name="voltage">
           <param name="initial_value">0.0</param>
@@ -102,4 +102,49 @@
         </state_interface>
       </sensor>
+      <sensor name="base_scan">
+        <state_interface name="range_min">
+          <param name="initial_value">0.120</param>
+        </state_interface>
+        <state_interface name="range_max">
+          <param name="initial_value">3.5</param>
+        </state_interface>
+        <state_interface name="angle_min">
+          <param name="initial_value">0.0</param>
+        </state_interface>
+        <state_interface name="angle_max">
+          <param name="initial_value">6.28319</param>
+        </state_interface>
+      </sensor>
+      <sensor name="line_laser">
+        <state_interface name="range_min">
+          <param name="initial_value">0.05</param>
+        </state_interface>
+        <state_interface name="range_max">
+          <param name="initial_value">2.0</param>
+        </state_interface>
+        <state_interface name="angle_min">
+          <param name="initial_value">-0.8</param>
+        </state_interface>
+        <state_interface name="angle_max">
+          <param name="initial_value">0.5</param>
+        </state_interface>
+      </sensor>
+      <sensor name="tof_camera">
+        <state_interface name="image_width">
+          <param name="initial_value">640</param>
+        </state_interface>
+        <state_interface name="image_height">
+          <param name="initial_value">480</param>
+        </state_interface>
+        <state_interface name="horizontal_fov">
+          <param name="initial_value">1.0</param>
+        </state_interface>
+        <state_interface name="near_clip">
+          <param name="initial_value">0.05</param>
+        </state_interface>
+        <state_interface name="far_clip">
+          <param name="initial_value">2.0</param>
+        </state_interface>
+      </sensor> -->
       <!--
       <joint name="${prefix}joint1">
