Commit message: sensors

File: src/turtlebot3_manipulation/turtlebot3_manipulation_description/urdf/custom_four_wheel_base.urdf.xacro (robot description, xacro)
@@ -2,12 +2,12 @@
 <robot xmlns:xacro="http://www.ros.org/wiki/xacro">
   <xacro:macro name="custom_four_wheel_base" params="prefix">
-    <!-- 标量变量 -->
     <xacro:property name="chassis_zero_height" value="0.09" />
-    <xacro:property name="chassis_length" value="0.41" />
-    <xacro:property name="chassis_width" value="0.4" />
+    <xacro:property name="chassis_length" value="0.3" />
+    <xacro:property name="chassis_width" value="0.25" />
     <xacro:property name="chassis_height" value="0.2" />
+    <xacro:property name="driver_radius" value="0.0675" />
+    <xacro:property name="driver_thickness" value="0.03" />
     <xacro:property name="driver_x_offset" value="-0.15" />
-    <xacro:property name="driver_y_offset" value="0.19" />
-    <xacro:property name="driver_radius" value="0.0675" />
+    <xacro:property name="driver_y_offset" value="${(chassis_width-driver_thickness)/2}" />
     <xacro:property name="caster_x_offset" value="0.15" />
     <xacro:property name="caster_y_offset" value="0.08" />
@@ -16,5 +16,17 @@
     <xacro:property name="chassis_heart_y_offset" value="0" />
     <xacro:property name="chassis_heart_z_offset" value="-0.05" />
+    <xacro:arg name="tof_x" default="${chassis_length/2}" />    <!-- ToF相机X位置 -->
+    <xacro:arg name="tof_y" default="0" />      <!-- ToF相机Y位置 -->
+    <xacro:arg name="tof_z" default="0.2" />   <!-- ToF相机传感器Z位置 -->
+    <xacro:arg name="line_x" default="0" />  <!-- 线激光X位置 -->
+    <xacro:arg name="line_y" default="${chassis_width/2}" />    <!-- 线激光Y位置 -->
+    <xacro:arg name="line_z" default="0.1" /> <!-- 线激光Z位置 -->
+    <xacro:arg name="line_mid_x" default="${chassis_length/2}" />  <!-- 线激光X位置 -->
+    <xacro:arg name="line_mid_rot_y" default="0.2" />
+    <xacro:arg name="line_mid_z" default="0.15" /> <!-- 线激光Z位置 -->
     <xacro:property name="caster_z_offset" value="${driver_radius - caster_radius}" />
+    <!-- 编码器尺寸 -->
+    <xacro:property name="encoder_radius" value="0.02" />
+    <xacro:property name="encoder_length" value="0.01" />
     <xacro:property
     name="meshes_file_direction"
@@ -26,5 +38,5 @@
       <parent link="${prefix}base_footprint"/>
       <child link="${prefix}base_link"/>
-      <origin xyz="0.0 0.0 ${driver_radius}" rpy="0 0 0"/>
+      <origin xyz="0 0 ${driver_radius}" rpy="0 0 0"/>
     </joint>
     <link name="${prefix}base_link">
@@ -78,5 +90,5 @@
         <origin xyz="0 0 0" rpy="0 0 0"/>
         <geometry>
-          <cylinder radius="${driver_radius}" length="0.03"/>
+          <cylinder radius="${driver_radius}" length="${driver_thickness}"/>
         </geometry>
         <material name="black"/>
@@ -85,5 +97,5 @@
         <origin xyz="0 0 0" rpy="0 0 0"/>
         <geometry>
-          <cylinder radius="${driver_radius}" length="0.03"/>
+          <cylinder radius="${driver_radius}" length="${driver_thickness}"/>
         </geometry>
       </collision>
@@ -96,4 +108,25 @@
       </inertial>
     </link>
+    <!-- 左侧编码器 -->
+    <joint name="${prefix}wheel_left_encoder_joint" type="fixed">
+      <parent link="${prefix}wheel_left_link"/>
+      <child link="${prefix}wheel_left_encoder_link"/>
+      <origin xyz="0 0 -0.015" rpy="0 0 0"/> <!-- 位于轮子中心 -->
+    </joint>
+    <link name="${prefix}wheel_left_encoder_link">
+      <visual>
+        <origin xyz="0 0 0" rpy="0 0 0"/>
+        <geometry>
+          <cylinder radius="${encoder_radius}" length="${encoder_length}"/>
+        </geometry>
+        <material name="yellow">
+          <color rgba="1 1 0 1"/> <!-- 黄色编码器 -->
+        </material>
+      </visual>
+      <inertial>
+        <mass value="0.01"/>
+        <inertia ixx="0.000001" ixy="0" ixz="0" iyy="0.000001" iyz="0" izz="0.000001"/>
+      </inertial>
+    </link>
     <!-- Right drive wheel -->
     <joint name="${prefix}wheel_right_joint" type="continuous">
@@ -107,5 +140,5 @@
         <origin xyz="0 0 0" rpy="0 0 0"/>
         <geometry>
-          <cylinder radius="${driver_radius}" length="0.03"/>
+          <cylinder radius="${driver_radius}" length="${driver_thickness}"/>
         </geometry>
         <material name="black"/>
@@ -114,5 +147,5 @@
         <origin xyz="0 0 0" rpy="0 0 0"/>
         <geometry>
-          <cylinder radius="${driver_radius}" length="0.03"/>
+          <cylinder radius="${driver_radius}" length="${driver_thickness}"/>
         </geometry>
       </collision>
@@ -125,4 +158,25 @@
       </inertial>
     </link>
+    <!-- 右侧编码器 (对称位置) -->
+    <joint name="${prefix}wheel_right_encoder_joint" type="fixed">
+      <parent link="${prefix}wheel_right_link"/>
+      <child link="${prefix}wheel_right_encoder_link"/>
+      <origin xyz="0 0 0.015" rpy="0 0 0"/> <!-- 与左侧对称 -->
+    </joint>
+    <link name="${prefix}wheel_right_encoder_link">
+      <visual>
+        <origin xyz="0 0 0" rpy="0 0 0"/>
+        <geometry>
+          <cylinder radius="${encoder_radius}" length="${encoder_length}"/>
+        </geometry>
+        <material name="yellow">
+          <color rgba="1 1 0 1"/> <!-- 黄色编码器 -->
+        </material>
+      </visual>
+      <inertial>
+        <mass value="0.01"/>
+        <inertia ixx="0.000001" ixy="0" ixz="0" iyy="0.000001" iyz="0" izz="0.000001"/>
+      </inertial>
+    </link>
     <joint name="${prefix}caster_front_left_joint" type="fixed">
       <parent link="${prefix}base_link"/>
@@ -130,25 +184,10 @@
       <origin xyz="${caster_x_offset} ${caster_y_offset} 0" rpy="0 0 0"/>
     </joint>
-    <joint name="${prefix}caster_front_right_joint" type="fixed">
-      <parent link="${prefix}base_link"/>
-      <child link="${prefix}caster_front_right_link"/>
-      <origin xyz="${caster_x_offset} ${-caster_y_offset} 0" rpy="0 0 0"/>
-    </joint>
-    <joint name="${prefix}caster_connector_left_joint" type="fixed">
-      <parent link="${prefix}base_link"/>
-      <child link="${prefix}caster_connector_left_link"/>
-      <origin xyz="${caster_x_offset} ${caster_y_offset} 0" rpy="0 0 0"/>
-    </joint>
-    <joint name="${prefix}caster_connector_right_joint" type="fixed">
-      <parent link="${prefix}base_link"/>
-      <child link="${prefix}caster_connector_right_link"/>
-      <origin xyz="${caster_x_offset} ${-caster_y_offset} 0" rpy="0 0 0"/>
-    </joint>
-    <link name="${prefix}caster_connector_left_link">
+    <link name="${prefix}caster_front_left_link">
       <!-- 添加固定连杆 -->
       <visual>
-        <origin xyz="0 0 ${chassis_zero_height/2-caster_z_offset}" rpy="0 0 0"/>
-        <geometry>
-          <cylinder radius="0.005" length="${chassis_zero_height-2*caster_radius}"/>
+        <origin xyz="0 0 ${-caster_z_offset}" rpy="0 0 0"/>
+        <geometry>
+          <sphere radius="${caster_radius}"/>
         </geometry>
         <material name="black">
@@ -157,11 +196,11 @@
       </visual>
       <collision>
-        <origin xyz="0 0 ${chassis_zero_height/2-caster_z_offset}" rpy="0 0 0"/>
-        <geometry>
-          <cylinder radius="0.005" length="${chassis_zero_height-2*caster_radius}"/>
-        </geometry>
-      </collision>
-      <inertial>
-        <origin xyz="0 0 ${chassis_zero_height/2-caster_z_offset}" rpy="0 0 0"/>
+        <origin xyz="0 0 ${-caster_z_offset}" rpy="0 0 0"/>
+        <geometry>
+          <sphere radius="${caster_radius}"/>
+        </geometry>
+      </collision>
+      <inertial>
+        <origin xyz="0 0 ${-caster_z_offset}" rpy="0 0 0"/>
         <mass value="0.1"/>
         <inertia ixx="0.00001" ixy="0.0" ixz="0.0"
@@ -170,10 +209,15 @@
       </inertial>
     </link>
-    <link name="${prefix}caster_front_left_link">
+    <joint name="${prefix}caster_connector_left_joint" type="fixed">
+      <parent link="${prefix}base_link"/>
+      <child link="${prefix}caster_connector_left_link"/>
+      <origin xyz="${caster_x_offset} ${caster_y_offset} 0" rpy="0 0 0"/>
+    </joint>
+    <link name="${prefix}caster_connector_left_link">
       <!-- 添加固定连杆 -->
       <visual>
-        <origin xyz="0 0 ${-caster_z_offset}" rpy="0 0 0"/>
-        <geometry>
-          <sphere radius="${caster_radius}"/>
+        <origin xyz="0 0 ${chassis_zero_height/2-caster_z_offset}" rpy="0 0 0"/>
+        <geometry>
+          <cylinder radius="0.005" length="${chassis_zero_height-2*caster_radius}"/>
         </geometry>
         <material name="black">
@@ -182,11 +226,11 @@
       </visual>
       <collision>
-        <origin xyz="0 0 ${-caster_z_offset}" rpy="0 0 0"/>
-        <geometry>
-          <sphere radius="${caster_radius}"/>
-        </geometry>
-      </collision>
-      <inertial>
-        <origin xyz="0 0 ${-caster_z_offset}" rpy="0 0 0"/>
+        <origin xyz="0 0 ${chassis_zero_height/2-caster_z_offset}" rpy="0 0 0"/>
+        <geometry>
+          <cylinder radius="0.005" length="${chassis_zero_height-2*caster_radius}"/>
+        </geometry>
+      </collision>
+      <inertial>
+        <origin xyz="0 0 ${chassis_zero_height/2-caster_z_offset}" rpy="0 0 0"/>
         <mass value="0.1"/>
         <inertia ixx="0.00001" ixy="0.0" ixz="0.0"
@@ -195,10 +239,15 @@
       </inertial>
     </link>
-    <link name="${prefix}caster_connector_right_link">
+    <joint name="${prefix}caster_front_right_joint" type="fixed">
+      <parent link="${prefix}base_link"/>
+      <child link="${prefix}caster_front_right_link"/>
+      <origin xyz="${caster_x_offset} ${-caster_y_offset} 0" rpy="0 0 0"/>
+    </joint>
+    <link name="${prefix}caster_front_right_link">
       <!-- 添加固定连杆 -->
       <visual>
-        <origin xyz="0 0 ${chassis_zero_height/2-caster_z_offset}" rpy="0 0 0"/>
-        <geometry>
-          <cylinder radius="0.005" length="${chassis_zero_height-2*caster_radius}"/>
+        <origin xyz="0 0 ${-caster_z_offset}" rpy="0 0 0"/>
+        <geometry>
+          <sphere radius="${caster_radius}"/>
         </geometry>
         <material name="black">
@@ -207,11 +256,11 @@
       </visual>
       <collision>
-        <origin xyz="0 0 ${chassis_zero_height/2-caster_z_offset}" rpy="0 0 0"/>
-        <geometry>
-          <cylinder radius="0.005" length="${chassis_zero_height-2*caster_radius}"/>
-        </geometry>
-      </collision>
-      <inertial>
-        <origin xyz="0 0 ${chassis_zero_height/2-caster_z_offset}" rpy="0 0 0"/>
+        <origin xyz="0 0 ${-caster_z_offset}" rpy="0 0 0"/>
+        <geometry>
+          <sphere radius="${caster_radius}"/>
+        </geometry>
+      </collision>
+      <inertial>
+        <origin xyz="0 0 ${-caster_z_offset}" rpy="0 0 0"/>
         <mass value="0.1"/>
         <inertia ixx="0.00001" ixy="0.0" ixz="0.0"
@@ -220,10 +269,15 @@
       </inertial>
     </link>
-    <link name="${prefix}caster_front_right_link">
+    <joint name="${prefix}caster_connector_right_joint" type="fixed">
+      <parent link="${prefix}base_link"/>
+      <child link="${prefix}caster_connector_right_link"/>
+      <origin xyz="${caster_x_offset} ${-caster_y_offset} 0" rpy="0 0 0"/>
+    </joint>
+    <link name="${prefix}caster_connector_right_link">
       <!-- 添加固定连杆 -->
       <visual>
-        <origin xyz="0 0 ${-caster_z_offset}" rpy="0 0 0"/>
-        <geometry>
-          <sphere radius="${caster_radius}"/>
+        <origin xyz="0 0 ${chassis_zero_height/2-caster_z_offset}" rpy="0 0 0"/>
+        <geometry>
+          <cylinder radius="0.005" length="${chassis_zero_height-2*caster_radius}"/>
         </geometry>
         <material name="black">
@@ -232,11 +286,11 @@
       </visual>
       <collision>
-        <origin xyz="0 0 ${-caster_z_offset}" rpy="0 0 0"/>
-        <geometry>
-          <sphere radius="${caster_radius}"/>
-        </geometry>
-      </collision>
-      <inertial>
-        <origin xyz="0 0 ${-caster_z_offset}" rpy="0 0 0"/>
+        <origin xyz="0 0 ${chassis_zero_height/2-caster_z_offset}" rpy="0 0 0"/>
+        <geometry>
+          <cylinder radius="0.005" length="${chassis_zero_height-2*caster_radius}"/>
+        </geometry>
+      </collision>
+      <inertial>
+        <origin xyz="0 0 ${chassis_zero_height/2-caster_z_offset}" rpy="0 0 0"/>
         <mass value="0.1"/>
         <inertia ixx="0.00001" ixy="0.0" ixz="0.0"
@@ -288,36 +342,93 @@
       </inertial>
     </link>
-    <joint name="${prefix}camera_joint" type="fixed">
-      <parent link="${prefix}base_link"/>
-      <child link="${prefix}camera_link"/>
-      <origin xyz="${chassis_length/2+0.01} 0 ${chassis_zero_height-driver_radius+chassis_height-0.01}" rpy="0 0 0"/>
-    </joint>
-    <link name="${prefix}camera_link">
-      <visual>
-        <origin xyz="0 0 0" rpy="0 0 0"/>
-        <geometry>
-          <box size="0.02 0.03 0.02"/>
-        </geometry>
-        <material name="dark"/>
-      </visual>
-      <collision>
-        <origin xyz="0 0 0" rpy="0 0 0"/>
-        <geometry>
-          <box size="0.02 0.03 0.02"/>
-        </geometry>
-      </collision>
-    </link>
-    <joint name="${prefix}camera_rgb_joint" type="fixed">
-      <parent link="${prefix}camera_link"/>
-      <child link="${prefix}camera_rgb_frame"/>
-      <origin xyz="0 0 0" rpy="0 0 0"/>
-    </joint>
-    <link name="${prefix}camera_rgb_frame"/>
-    <joint name="${prefix}camera_rgb_optical_joint" type="fixed">
-      <parent link="${prefix}camera_rgb_frame"/>
-      <child link="${prefix}camera_rgb_optical_frame"/>
+    <!-- 左线激光传感器 - 增强可视化 -->
+    <joint name="${prefix}line_laser_left_joint" type="fixed">
+      <parent link="${prefix}base_link"/>
+      <child link="${prefix}line_laser_left"/>
+      <origin xyz="$(arg line_x) $(arg line_y) $(arg line_z)" rpy="1.57 0 1.57"/>
+    </joint>
+    <link name="${prefix}line_laser_left">
+      <visual>
+        <origin xyz="0 0 0" rpy="0 0 0"/> <!--  -->
+        <geometry>
+          <cylinder radius="0.02" length="0.02"/> <!-- 使用细长圆柱体 -->
+        </geometry>
+        <material name="red_transparent">
+          <color rgba="1 0 0 0.9"/> <!-- 更鲜艳的红色 -->
+        </material>
+      </visual>
+      <inertial>
+        <mass value="0.02"/>
+        <inertia ixx="0.00001" ixy="0" ixz="0" iyy="0.00001" iyz="0" izz="0.00001"/>
+      </inertial>
+    </link>
+    <!-- 中线激光传感器 - 增强可视化 -->
+    <joint name="${prefix}line_laser_mid_joint" type="fixed">
+      <parent link="${prefix}base_link"/>
+      <child link="${prefix}line_laser_mid"/>
+      <origin xyz="$(arg line_mid_x) 0 $(arg line_mid_z)" rpy="0 $(arg line_mid_rot_y) 0"/>
+    </joint>
+    <link name="${prefix}line_laser_mid">
+      <visual>
+        <origin xyz="0 0 0" rpy="0 0 0"/> <!--  -->
+        <geometry>
+          <cylinder radius="0.02" length="0.02"/> <!-- 使用细长圆柱体 -->
+        </geometry>
+        <material name="red_transparent">
+          <color rgba="1 0 0 0.9"/> <!-- 更鲜艳的红色 -->
+        </material>
+      </visual>
+      <inertial>
+        <mass value="0.02"/>
+        <inertia ixx="0.00001" ixy="0" ixz="0" iyy="0.00001" iyz="0" izz="0.00001"/>
+      </inertial>
+    </link>
+    <!-- 右线激光传感器 - 增强可视化 -->
+    <joint name="${prefix}line_laser_right_joint" type="fixed">
+      <parent link="${prefix}base_link"/>
+      <child link="${prefix}line_laser_right"/>
+      <origin xyz="$(arg line_x) -$(arg line_y) $(arg line_z)" rpy="1.57 0 -1.57"/>
+    </joint>
+    <link name="${prefix}line_laser_right">
+      <visual>
+        <origin xyz="0 0 0" rpy="0 0 0"/> <!--  -->
+        <geometry>
+          <cylinder radius="0.02" length="0.02"/> <!-- 使用细长圆柱体 -->
+        </geometry>
+        <material name="red_transparent">
+          <color rgba="1 0 0 0.9"/> <!-- 更鲜艳的红色 -->
+        </material>
+      </visual>
+      <inertial>
+        <mass value="0.02"/>
+        <inertia ixx="0.00001" ixy="0" ixz="0" iyy="0.00001" iyz="0" izz="0.00001"/>
+      </inertial>
+    </link>
+    <!-- 3D ToF深度相机 -->
+    <joint name="${prefix}tof_camera_joint" type="fixed">
+      <parent link="${prefix}base_link"/>
+      <child link="${prefix}tof_camera"/>
+      <origin xyz="$(arg tof_x) $(arg tof_y) $(arg tof_z)" rpy="0 0 0"/>
+    </joint>
+    <link name="${prefix}tof_camera">
+      <visual>
+        <geometry>
+          <box size="0.03 0.03 0.02"/>
+        </geometry>
+        <material name="camera">
+          <color rgba="0.3 0.3 0.3 1.0"/>
+        </material>
+      </visual>
+      <inertial>
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
File: src/turtlebot3_manipulation/turtlebot3_manipulation_description/urdf/fhbot.urdf.xacro (robot description, xacro)
@@ -39,5 +39,5 @@
     use_fake_hardware="$(arg use_fake_hardware)"
     fake_sensor_commands="$(arg fake_sensor_commands)"/>
-  <!--加载gazebo的ros2控制插件和参数配置文件 -->
+  <!--加载gazebo的ros2控制器管理器配置文件 -->
   <gazebo>
     <plugin name="gazebo_ros2_control" filename="libgazebo_ros2_control.so">

Commit message: mapping

File: src/turtlebot3_manipulation/turtlebot3_manipulation_description/gazebo/custom_four_wheel_base.gazebo.xacro (robot description, xacro)
@@ -2,5 +2,5 @@
 <robot xmlns:xacro="http://ros.org/wiki/xacro">
   <xacro:macro name="custom_four_wheel_base_gazebo" params="prefix">
-    <xacro:property name="laser_visual"      value="false"/>
+    <xacro:property name="laser_visual"      value="true"/>
     <xacro:property name="imu_visual"        value="true"/>
     <xacro:property name="line_laser_visual" value="true"/>
@@ -195,5 +195,5 @@
           <ros>
             <namespace></namespace>
-            <remapping>~/out:=base_scan</remapping>
+            <remapping>~/out:=scan</remapping>
           </ros>
           <output_type>sensor_msgs/LaserScan</output_type>

File: src/turtlebot3_manipulation/turtlebot3_manipulation_description/urdf/custom_four_wheel_base.urdf.xacro (robot description, xacro)
@@ -3,6 +3,6 @@
   <xacro:macro name="custom_four_wheel_base" params="prefix">
     <xacro:property name="chassis_zero_height" value="0.09" />
-    <xacro:property name="chassis_length" value="0.3" />
-    <xacro:property name="chassis_width" value="0.25" />
+    <xacro:property name="chassis_length" value="0.35" />
+    <xacro:property name="chassis_width" value="0.41" />
     <xacro:property name="chassis_height" value="0.2" />
     <xacro:property name="driver_radius" value="0.0675" />

Commit message: amcl + imu

File: src/turtlebot3_manipulation/turtlebot3_manipulation_description/gazebo/custom_four_wheel_base.gazebo.xacro (robot description, xacro)
@@ -4,5 +4,7 @@
     <xacro:property name="laser_visual"      value="true"/>
     <xacro:property name="imu_visual"        value="true"/>
-    <xacro:property name="line_laser_visual" value="true"/>
+    <xacro:property name="left_line_laser_visual" value="false"/>
+    <xacro:property name="mid_line_laser_visual" value="true"/>
+    <xacro:property name="right_line_laser_visual" value="false"/>
     <xacro:property name="tof_camera_visual" value="true"/>
     <xacro:property name="base_laser_samples" value="360"/>
@@ -99,8 +101,10 @@
       <plugin name='diff_drive' filename='libgazebo_ros_diff_drive.so'>
         <ros>
-          <namespace></namespace>
+          <namespace>/</namespace>
           <remapping>cmd_vel:=cmd_vel</remapping>
           <remapping>odom:=odom</remapping>
         </ros>
+        <update_rate>100.0</update_rate>  <!-- 限制为30Hz -->
+        <publish_rate>100.0</publish_rate> <!-- 发布频率限制 -->
         <left_joint>wheel_left_joint</left_joint>
         <right_joint>wheel_right_joint</right_joint>
@@ -165,4 +169,11 @@
           </linear_acceleration>
         </imu>
+        <plugin name="gazebo_ros_imu_controller" filename="libgazebo_ros_imu_sensor.so">
+          <ros>
+            <namespace></namespace>
+            <remapping>~/out:=imu</remapping>
+          </ros>
+          <initial_orientation_as_reference>false</initial_orientation_as_reference>
+        </plugin>
       </sensor>
     </gazebo>
@@ -208,5 +219,5 @@
         <always_on>true</always_on>
         <update_rate>${line_laser_rate}</update_rate>
-        <visualize>${line_laser_visual}</visualize>
+        <visualize>${left_line_laser_visual}</visualize>
         <ray>
           <scan>
@@ -251,5 +262,5 @@
         <always_on>true</always_on>
         <update_rate>${line_laser_rate}</update_rate>
-        <visualize>${line_laser_visual}</visualize>
+        <visualize>${mid_line_laser_visual}</visualize>
         <ray>
           <scan>
@@ -294,5 +305,5 @@
         <always_on>true</always_on>
         <update_rate>${line_laser_rate}</update_rate>
-        <visualize>${line_laser_visual}</visualize>
+        <visualize>${right_line_laser_visual}</visualize>
         <ray>
           <scan>

File: src/turtlebot3_manipulation/turtlebot3_manipulation_description/urdf/custom_four_wheel_base.urdf.xacro (robot description, xacro)
@@ -3,7 +3,7 @@
   <xacro:macro name="custom_four_wheel_base" params="prefix">
     <xacro:property name="chassis_zero_height" value="0.09" />
-    <xacro:property name="chassis_length" value="0.35" />
+    <xacro:property name="chassis_length" value="0.4" />
     <xacro:property name="chassis_width" value="0.41" />
-    <xacro:property name="chassis_height" value="0.2" />
+    <xacro:property name="chassis_height" value="0.35" />
     <xacro:property name="driver_radius" value="0.0675" />
     <xacro:property name="driver_thickness" value="0.03" />
@@ -18,11 +18,11 @@
     <xacro:arg name="tof_x" default="${chassis_length/2}" />    <!-- ToF相机X位置 -->
     <xacro:arg name="tof_y" default="0" />      <!-- ToF相机Y位置 -->
-    <xacro:arg name="tof_z" default="0.2" />   <!-- ToF相机传感器Z位置 -->
+    <xacro:arg name="tof_z" default="${chassis_height}" />   <!-- ToF相机传感器Z位置 -->
     <xacro:arg name="line_x" default="0" />  <!-- 线激光X位置 -->
     <xacro:arg name="line_y" default="${chassis_width/2}" />    <!-- 线激光Y位置 -->
-    <xacro:arg name="line_z" default="0.1" /> <!-- 线激光Z位置 -->
+    <xacro:arg name="line_z" default="0.2" /> <!-- 线激光Z位置 -->
     <xacro:arg name="line_mid_x" default="${chassis_length/2}" />  <!-- 线激光X位置 -->
-    <xacro:arg name="line_mid_rot_y" default="0.2" />
-    <xacro:arg name="line_mid_z" default="0.15" /> <!-- 线激光Z位置 -->
+    <xacro:arg name="line_mid_rot_y" default="0.785" />
+    <xacro:arg name="line_mid_z" default="0.25" /> <!-- 线激光Z位置 -->
     <xacro:property name="caster_z_offset" value="${driver_radius - caster_radius}" />
     <!-- 编码器尺寸 -->
