Commit message: base_link

File: src/turtlebot3_manipulation/turtlebot3_manipulation_description/gazebo/custom_four_wheel_base.gazebo.xacro (robot description, xacro)
@@ -117,5 +117,5 @@
         <publish_wheel_tf>false</publish_wheel_tf>
         <odometry_frame>odom</odometry_frame>
-        <robot_base_frame>base_footprint</robot_base_frame>
+        <robot_base_frame>base_link</robot_base_frame>
       </plugin>
     </gazebo>

File: src/turtlebot3_manipulation/turtlebot3_manipulation_description/gazebo/turtlebot3_waffle_pi.gazebo.xacro (robot description, xacro)
@@ -75,5 +75,5 @@
       <publish_wheel_tf>false</publish_wheel_tf>
       <odometry_frame>odom</odometry_frame>
-      <robot_base_frame>base_footprint</robot_base_frame>
+      <robot_base_frame>base_link</robot_base_frame>
     </plugin>
   </gazebo>

File: src/turtlebot3_manipulation/turtlebot3_manipulation_description/urdf/custom_four_wheel_base.urdf.xacro (robot description, xacro)
@@ -33,12 +33,12 @@
     value="package://turtlebot3_manipulation_description/meshes/turtlebot3_waffle_pi"/>
     <!-- Base footprint -->
-    <link name="${prefix}base_footprint"/>
+    <link name="${prefix}base_link"/>
     <!-- Base link -->
     <joint name="${prefix}base_joint" type="fixed">
-      <parent link="${prefix}base_footprint"/>
-      <child link="${prefix}base_link"/>
-      <origin xyz="0 0 ${driver_radius}" rpy="0 0 0"/>
-    </joint>
-    <link name="${prefix}base_link">
+      <parent link="${prefix}base_link"/>
+      <child link="${prefix}base_link_temp"/>
+      <origin xyz="${-driver_x_offset} 0 ${driver_radius}" rpy="0 0 0"/>
+    </joint>
+    <link name="${prefix}base_link_temp">
       <visual>
         <origin xyz="0 0 ${chassis_zero_height+chassis_height/2-driver_radius}" rpy="0 0 0"/>
@@ -65,5 +65,5 @@
     </link>
     <joint name="${prefix}center_of_mass_joint" type="fixed">
-      <parent link="${prefix}base_link"/>
+      <parent link="${prefix}base_link_temp"/>
       <child link="${prefix}center_of_mass_link"/>
       <origin xyz="${chassis_heart_x_offset} ${chassis_heart_y_offset} ${chassis_zero_height+chassis_height/2-driver_radius+chassis_heart_z_offset}" rpy="0 0 0"/>
@@ -81,5 +81,5 @@
     <!-- Left drive wheel -->
     <joint name="${prefix}wheel_left_joint" type="continuous">
-      <parent link="${prefix}base_link"/>
+      <parent link="${prefix}base_link_temp"/>
       <child link="${prefix}wheel_left_link"/>
       <origin xyz="${driver_x_offset} ${driver_y_offset} 0" rpy="-1.57 0 0"/>
@@ -131,5 +131,5 @@
     <!-- Right drive wheel -->
     <joint name="${prefix}wheel_right_joint" type="continuous">
-      <parent link="${prefix}base_link"/>
+      <parent link="${prefix}base_link_temp"/>
       <child link="${prefix}wheel_right_link"/>
       <origin xyz="${driver_x_offset} ${-driver_y_offset} 0" rpy="-1.57 0 0"/>
@@ -180,5 +180,5 @@
     </link>
     <joint name="${prefix}caster_front_left_joint" type="fixed">
-      <parent link="${prefix}base_link"/>
+      <parent link="${prefix}base_link_temp"/>
       <child link="${prefix}caster_front_left_link"/>
       <origin xyz="${caster_x_offset} ${caster_y_offset} 0" rpy="0 0 0"/>
@@ -210,5 +210,5 @@
     </link>
     <joint name="${prefix}caster_connector_left_joint" type="fixed">
-      <parent link="${prefix}base_link"/>
+      <parent link="${prefix}base_link_temp"/>
       <child link="${prefix}caster_connector_left_link"/>
       <origin xyz="${caster_x_offset} ${caster_y_offset} 0" rpy="0 0 0"/>
@@ -240,5 +240,5 @@
     </link>
     <joint name="${prefix}caster_front_right_joint" type="fixed">
-      <parent link="${prefix}base_link"/>
+      <parent link="${prefix}base_link_temp"/>
       <child link="${prefix}caster_front_right_link"/>
       <origin xyz="${caster_x_offset} ${-caster_y_offset} 0" rpy="0 0 0"/>
@@ -270,5 +270,5 @@
     </link>
     <joint name="${prefix}caster_connector_right_joint" type="fixed">
-      <parent link="${prefix}base_link"/>
+      <parent link="${prefix}base_link_temp"/>
       <child link="${prefix}caster_connector_right_link"/>
       <origin xyz="${caster_x_offset} ${-caster_y_offset} 0" rpy="0 0 0"/>
@@ -300,5 +300,5 @@
     </link>
     <joint name="${prefix}imu_joint" type="fixed">
-      <parent link="${prefix}base_link"/>
+      <parent link="${prefix}base_link_temp"/>
       <child link="${prefix}imu_link"/>
       <origin xyz="0.0 0 ${chassis_zero_height-driver_radius-0.01}" rpy="0 0 0"/>
@@ -316,5 +316,5 @@
     </link>
     <joint name="${prefix}scan_joint" type="fixed">
-      <parent link="${prefix}base_link"/>
+      <parent link="${prefix}base_link_temp"/>
       <child link="${prefix}base_scan"/>
       <origin xyz="${chassis_length/2-0.08} 0 ${chassis_zero_height-driver_radius+chassis_height+0.01}" rpy="0 0 0"/>
@@ -344,5 +344,5 @@
     <!-- 左线激光传感器 - 增强可视化 -->
     <joint name="${prefix}line_laser_left_joint" type="fixed">
-      <parent link="${prefix}base_link"/>
+      <parent link="${prefix}base_link_temp"/>
       <child link="${prefix}line_laser_left"/>
       <origin xyz="$(arg line_x) $(arg line_y) $(arg line_z)" rpy="1.57 0 1.57"/>
@@ -365,5 +365,5 @@
     <!-- 中线激光传感器 - 增强可视化 -->
     <joint name="${prefix}line_laser_mid_joint" type="fixed">
-      <parent link="${prefix}base_link"/>
+      <parent link="${prefix}base_link_temp"/>
       <child link="${prefix}line_laser_mid"/>
       <origin xyz="$(arg line_mid_x) 0 $(arg line_mid_z)" rpy="0 $(arg line_mid_rot_y) 0"/>
@@ -386,5 +386,5 @@
     <!-- 右线激光传感器 - 增强可视化 -->
     <joint name="${prefix}line_laser_right_joint" type="fixed">
-      <parent link="${prefix}base_link"/>
+      <parent link="${prefix}base_link_temp"/>
       <child link="${prefix}line_laser_right"/>
       <origin xyz="$(arg line_x) -$(arg line_y) $(arg line_z)" rpy="1.57 0 -1.57"/>
@@ -407,5 +407,5 @@
     <!-- 3D ToF深度相机 -->
     <joint name="${prefix}tof_camera_joint" type="fixed">
-      <parent link="${prefix}base_link"/>
+      <parent link="${prefix}base_link_temp"/>
       <child link="${prefix}tof_camera"/>
       <origin xyz="$(arg tof_x) $(arg tof_y) $(arg tof_z)" rpy="0 0 0"/>

File: src/turtlebot3_manipulation/turtlebot3_manipulation_description/urdf/turtlebot3_waffle_pi.urdf.xacro (robot description, xacro)
@@ -10,7 +10,7 @@
     name="meshes_file_direction"
     value="package://turtlebot3_manipulation_description/meshes/turtlebot3_waffle_pi"/>
-  <link name="${prefix}base_footprint"/>
+  <link name="${prefix}base_link"/>
   <joint name="${prefix}base_joint" type="fixed">
-    <parent link="${prefix}base_footprint"/>
+    <parent link="${prefix}base_link"/>
     <child link="${prefix}base_link" />
     <origin xyz="0 0 0.010" rpy="0 0 0"/>
